File: PCB/Alarm clock pcb.kicad_pcb (KiCad board)
At the start: 2 copper layers, 110.5 x 55.1 mm, 11 parts, among them U2 MCU_Seeed_XIAO_RP2040

Commit message: Add new folder or changes
Routing:
- added copper zone on B.Cu, net (none)
- added copper zone on F.Cu, net (none)
- removed copper zone on B.Cu, net GND
- removed copper zone on F.Cu, net GND
Other:
- board size 110.5 x 55.1 mm -> 117.5 x 57.5 mm
Changed lines of the file:
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@@
 	)
 	(gr_rect
-		(start 154.4 73.325)
-		(end 264.9 128.4)
+		(start 151 72)
+		(end 268.5 129.5)
 		(stroke
 			(width 0.05)
@@
 	)
 	(gr_circle
-		(center 158.15 76.45)
-		(end 156.4 76.475)
+		(center 155.5 76.5)
+		(end 157.25 76.5)
 		(stroke
 			(width 0.05)
@@
 	)
 	(gr_circle
-		(center 158.15 125.35)
-		(end 157.625 123.675)
+		(center 155.5 125)
+		(end 157.25 125)
 		(stroke
 			(width 0.05)
@@
 	)
 	(gr_circle
-		(center 261.175 78.475)
-		(end 262.875 78.025)
+		(center 264 125)
+		(end 265.75 125)
 		(stroke
 			(width 0.05)
@@
 	)
 	(gr_circle
-		(center 261.175 125.2)
-		(end 262.425 123.95)
+		(center 264.5 76.5)
+		(end 266.25 76.5)
 		(stroke
 			(width 0.05)
@@
 	)
 	(zone
-		(net "GND")
 		(layers "F.Cu" "B.Cu")
 		(hatch edge 0.5)
@@
 			(thermal_gap 0.5)
 			(thermal_bridge_width 0.5)
-			(island_removal_mode 0)
+			(island_removal_mode 1)
 		)
 		(polygon
 			(pts
-				(xy 275.075 67.65) (xy 148.1 67.65) (xy 148.1 134.15) (xy 150.55 136.6) (xy 270.35 136.6) (xy 275.075 131.875)
+				(xy 274.5 64) (xy 143 64) (xy 142.5 64.5) (xy 142.5 139) (xy 274.5 139)
 			)
 		)
